File: hardware/battery_charger_devboard_multi/battery_charger_devboard_multi.kicad_sch (KiCad schematic)
At the start: 125 parts, among them J1 NTC1, J10 BAT, J11 CHRG3, J12 CHRG2, J13 BAT_OUT, J14 CHRG4, J15 NTC2, J16 PGM, J17 BAT4, J18 VIN, J19 OUT, J2 Program, J20 BAT_OUT2, J3 USB-C PD, J4 BAT1, J5 CHRG1, J6 MCU, J7 BAT2, J8 BAT2, J9 OUT, Q1 AO3401A, Q2 AO3401A, Q3 AO3401A, Q4 AO3401A, Q5 AO3401A, SW1 Boot, SW2 On, U1 AW32001E, U2 CH224Q, U3 USBLC6-2SC6, U4 HT75xx-1-SOT89, U5 APW7261, U6 AW32257, U7 CH32V003F4U6, U8 TP5100

Commit message: Added documentation
Parts:
- R26, R27: symbol Device:R -> Device:R_Small
Other:
- note added: "Battery reverse polarity protection"
- moved on the sheet: Q5, R26, R27
Changed lines of the file:
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@@
 		(comment 2 "https://github.com/Subjective-Reality-Labs/")
 	)
+	(rectangle
+		(start 154.94 65.405)
+		(end 188.595 85.09)
+		(stroke
+			(width 0)
+			(type dash)
+		)
+		(fill
+			(type none)
+		)
+	)
 	(text "R_{SNS} (R13) selection per datasheet:\n56m, 68m, 100m\nThe higher the value, the lower is charging current."
 		(exclude_from_sim no)
@@
 		)
 	)
+	(text "Battery reverse polarity\nprotection"
+		(exclude_from_sim no)
+		(at 155.448 68.072 0)
+		(effects
+			(font
+				(size 1.27 1.27)
+			)
+			(justify left)
+		)
+	)
 	(text "3 of 4 charge ICs use internal buck converter to generate output voltage.\nThis requires a suitable inductor. I_{sat} of selected indutor has to be bigger than\npeak current of the buck converter that can be calculated using this formula:\nI_{peak} = I_{out} + ((V_{in}-v_{out})*D)/(2*L*freq))\nwhere D is duty cycle: D = V_{out}/V_{in}\nAW32257 maximum charging current is 2.5A @1.5MHz,\nAPW7261 is 1.5A @3MHz,\nTP5100 is 2A @800kHz."
 		(exclude_from_sim no)
@@
 	)
 	(junction
+		(at 162.56 91.44)
+		(diameter 0)
+		(color 0 0 0 0)
+	)
+	(junction
 		(at 60.96 21.59)
 		(diameter 0)
@@
 	)
 	(junction
-		(at 168.91 83.82)
-		(diameter 0)
-		(color 0 0 0 0)
-	)
-	(junction
 		(at 25.4 60.96)
 		(diameter 0)
@@
 	)
 	(junction
-		(at 162.56 91.44)
-		(diameter 0)
-		(color 0 0 0 0)
-	)
-	(junction
 		(at 95.25 167.64)
 		(diameter 0)
@@
 	(wire
 		(pts
-			(xy 168.91 83.82) (xy 168.91 78.74)
+			(xy 168.91 78.74) (xy 168.91 88.9)
 		)
 		(stroke
@@
 	(wire
 		(pts
+			(xy 156.21 78.74) (xy 157.48 78.74)
+		)
+		(stroke
+			(width 0)
+			(type default)
+		)
+	)
+	(wire
+		(pts
 			(xy 31.75 177.8) (xy 40.64 177.8)
 		)
@@
 	(wire
 		(pts
+			(xy 254 27.94) (xy 254 29.21)
+		)
+		(stroke
+			(width 0)
+			(type default)
+		)
+	)
+	(wire
+		(pts
 			(xy 222.25 135.89) (xy 226.06 135.89)
 		)
@@
 	(wire
 		(pts
-			(xy 156.21 83.82) (xy 157.48 83.82)
-		)
-		(stroke
-			(width 0)
-			(type default)
-		)
-	)
-	(wire
-		(pts
 			(xy 100.33 21.59) (xy 101.6 21.59)
 		)
@@
 	(wire
 		(pts
+			(xy 162.56 91.44) (xy 168.91 91.44)
+		)
+		(stroke
+			(width 0)
+			(type default)
+		)
+	)
+	(wire
+		(pts
 			(xy 66.04 142.24) (xy 67.31 142.24)
 		)
@@
 	(wire
 		(pts
-			(xy 167.64 83.82) (xy 168.91 83.82)
+			(xy 162.56 86.36) (xy 162.56 91.44)
 		)
 		(stroke
@@
 	(wire
 		(pts
+			(xy 167.64 78.74) (xy 168.91 78.74)
+		)
+		(stroke
+			(width 0)
+			(type default)
+		)
+	)
+	(wire
+		(pts
 			(xy 114.3 184.15) (xy 111.76 184.15)
 		)
@@
 	(wire
 		(pts
-			(xy 162.56 91.44) (xy 168.91 91.44)
-		)
-		(stroke
-			(width 0)
-			(type default)
-		)
-	)
-	(wire
-		(pts
 			(xy 281.94 118.11) (xy 281.94 146.05)
 		)
@@
 	(wire
 		(pts
-			(xy 168.91 83.82) (xy 168.91 88.9)
-		)
-		(stroke
-			(width 0)
-			(type default)
-		)
-	)
-	(wire
-		(pts
 			(xy 46.99 36.83) (xy 55.88 36.83)
 		)
@@
 	(wire
 		(pts
+			(xy 256.54 27.94) (xy 256.54 29.21)
+		)
+		(stroke
+			(width 0)
+			(type default)
+		)
+	)
+	(wire
+		(pts
 			(xy 33.02 127) (xy 33.02 128.27)
 		)
@@
 	(wire
 		(pts
-			(xy 156.21 88.9) (xy 156.21 83.82)
+			(xy 156.21 78.74) (xy 156.21 88.9)
 		)
 		(stroke
@@
 	(global_label "SCL"
 		(shape input)
-		(at 256.54 30.48 270)
+		(at 256.54 29.21 270)
 		(fields_autoplaced yes)
 		(effects
@@
 		)
 		(property "Intersheetrefs" "${INTERSHEET_REFS}"
-			(at 256.54 36.9728 90)
+			(at 256.54 35.7028 90)
 			(effects
 				(font
@@
 	(global_label "SDA"
 		(shape input)
-		(at 254 30.48 270)
+		(at 254 29.21 270)
 		(fields_autoplaced yes)
 		(effects
@@
 		)
 		(property "Intersheetrefs" "${INTERSHEET_REFS}"
-			(at 254 37.0333 90)
+			(at 254 35.7633 90)
 			(effects
 				(font
@@
 	(global_label "OUT_LOAD"
 		(shape input)
-		(at 144.78 77.47 0)
+		(at 144.78 77.47 90)
 		(fields_autoplaced yes)
 		(effects
@@
 		)
 		(property "Intersheetrefs" "${INTERSHEET_REFS}"
-			(at 157.0786 77.47 0)
+			(at 144.78 65.1714 90)
 			(effects
 				(font
@@
 	)
 	(symbol
-		(lib_id "Device:R")
-		(at 254 26.67 180)
+		(lib_name "R_Small_1")
+		(lib_id "Device:R_Small")
+		(at 254 25.4 180)
 		(unit 1)
 		(exclude_from_sim no)
@@
 		(dnp no)
 		(property "Reference" "R26"
-			(at 251.968 26.67 90)
+			(at 251.968 25.4 90)
 			(effects
 				(font
@@
 		)
 		(property "Value" "10K"
-			(at 254 26.67 90)
+			(at 254 25.4 90)
 			(effects
 				(font
@@
 		)
 		(property "Footprint" "Resistor_SMD:R_0402_1005Metric"
-			(at 255.778 26.67 90)
+			(at 254 25.4 0)
 			(effects
 				(font
@@
 		)
 		(property "Datasheet" "~"
-			(at 254 26.67 0)
+			(at 254 25.4 0)
 			(effects
 				(font
@@
 			)
 		)
-		(property "Description" "Resistor"
-			(at 254 26.67 0)
+		(property "Description" "Resistor, small symbol"
+			(at 254 25.4 0)
 			(effects
 				(font
@@
 		)
 		(property "LCSC" "C60490"
-			(at 254 26.67 90)
+			(at 254 25.4 90)
 			(effects
 				(font
@@
 	)
 	(symbol
-		(lib_id "Device:R")
-		(at 256.54 26.67 0)
+		(lib_name "R_Small_2")
+		(lib_id "Device:R_Small")
+		(at 256.54 25.4 0)
 		(mirror x)
 		(unit 1)
@@
 		(dnp no)
 		(property "Reference" "R27"
-			(at 258.572 26.67 90)
+			(at 258.572 25.4 90)
 			(effects
 				(font
@@
 		)
 		(property "Value" "10K"
-			(at 256.54 26.67 90)
+			(at 256.54 25.4 90)
 			(effects
 				(font
@@
 		)
 		(property "Footprint" "Resistor_SMD:R_0402_1005Metric"
-			(at 254.762 26.67 90)
+			(at 256.54 25.4 0)
 			(effects
 				(font
@@
 		)
 		(property "Datasheet" "~"
-			(at 256.54 26.67 0)
+			(at 256.54 25.4 0)
 			(effects
 				(font
@@
 			)
 		)
-		(property "Description" "Resistor"
-			(at 256.54 26.67 0)
+		(property "Description" "Resistor, small symbol"
+			(at 256.54 25.4 0)
 			(effects
 				(font
@@
 		)
 		(property "LCSC" "C60490"
-			(at 256.54 26.67 90)
+			(at 256.54 25.4 90)
 			(effects
 				(font
@@
 	(symbol
 		(lib_id "Transistor_FET:AO3401A")
-		(at 162.56 86.36 270)
+		(at 162.56 81.28 270)
 		(mirror x)
 		(unit 1)
@@
 		(dnp no)
 		(property "Reference" "Q5"
-			(at 163.7722 81.153 90)
+			(at 163.7722 76.073 90)
 			(effects
 				(font
@@
 		)
 		(property "Value" "AO3401A"
-			(at 158.75 78.994 90)
+			(at 158.75 73.914 90)
 			(effects
 				(font
@@
 		)
 		(property "Footprint" "Package_TO_SOT_SMD:SOT-23"
-			(at 160.655 81.28 0)
+			(at 160.655 76.2 0)
 			(effects
 				(font
@@
 		)
 		(property "Datasheet" "http://www.aosmd.com/pdfs/datasheet/AO3401A.pdf"
-			(at 158.75 81.28 0)
+			(at 158.75 76.2 0)
 			(effects
 				(font
@@
 		)
 		(property "Description" "-4.0A Id, -30V Vds, P-Channel MOSFET, SOT-23"
-			(at 162.56 86.36 0)
+			(at 162.56 81.28 0)
 			(effects
 				(font
@@
 		)
 		(property "LCSC" "C306862"
-			(at 162.56 86.36 90)
+			(at 162.56 81.28 90)
 			(effects
 				(font
